File: st225/20301/DigitalStepper.kicad_sch (KiCad schematic)
At the start: 74 parts, among them J3 POWER, J6 STEPPER, Q11 2N3906, Q12 2N3906, Q9 2N3906, Y1 ?MHz

Commit message: Numerous small changes, README updates
Parts:
- Y1: value ?MHz -> 2MHz
Changed lines of the file:
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@@
       (effects (font (size 1.27 1.27)))
     )
-    (property "Value" "?MHz" (at 176.53 64.77 0)
+    (property "Value" "2MHz" (at 176.53 64.77 0)
       (effects (font (size 1.27 1.27)))
     )

Commit message: st225 updates with more info
Connections:
- net START/~{RUN}: now reaches 5B1.14 (PC6), R50.2
Other:
- note added: "300ns"
- note added: "Microstepping hardware for recovery mode (often not installed)"
- note added: "Per-track microstep lookup table perhaps experimental feature? (not installed)"
Changed lines of the file:
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@@
     (stroke (width 0) (type default))
+  )
+  (rectangle (start 251.46 121.92) (end 326.39 198.12)
+    (stroke (width 0) (type dash))
+    (fill (type none))
+  )
+  (rectangle (start 276.86 40.64) (end 378.46 119.38)
+    (stroke (width 0) (type dash))
+    (fill (type none))
+  )
+  (text "Microstepping hardware\nfor recovery mode\n(often not installed)"
+    (at 320.04 48.26 0)
+    (effects (font (size 1.27 1.27)) (justify left bottom))
   )
   (text "This work is licensed under a Creative Commons\nAttribution-ShareAlike 4.0 International License.\nSee https://creativecommons.org/licenses/by-sa/4.0/.\n"
@@
     (effects (font (size 1.27 1.27)) (justify left bottom))
   )
+  (text "300ns" (at 22.86 102.87 0)
+    (effects (font (size 1.27 1.27)) (justify left bottom))
+  )
   (text "Reverse Engineered by Tube Time" (at 302.26 266.7 0)
+    (effects (font (size 1.27 1.27)) (justify left bottom))
+  )
+  (text "Per-track microstep lookup table\nperhaps experimental feature?\n(not installed)"
+    (at 292.1 129.54 0)
     (effects (font (size 1.27 1.27)) (justify left bottom))
   )
@@
     (effects (font (size 1.27 1.27)) (justify left bottom))
   )
+  (label "START{slash}~{RUN}" (at 260.35 201.93 0) (fields_autoplaced)
+    (effects (font (size 1.27 1.27)) (justify left bottom))
+  )
